Commit message: added xacro

File: src/my_robot_description/urdf/my_robot.urdf.xacro (robot description, xacro)
@@ -6,4 +6,15 @@
     <xacro:property name="wheel_radius" value="0.1" />
     <xacro:property name="wheel_length" value="0.05" />
+    <xacro:macro name="wheel_link" params="prefix">
+        <link name="${prefix}_wheel_link">
+            <visual>
+                <geometry>
+                    <cylinder radius="${wheel_radius}" length="${wheel_length}" />
+                </geometry>
+                <origin xyz="0 0 0" rpy="${pi/2.0} 0 0" />
+                <material name="grey" />
+            </visual>
+        </link>
+    </xacro:macro>
     <material name="blue">
         <color rgba="0 0 1 1" />
@@ -12,4 +23,6 @@
         <color rgba="0.5 0.5 0.5 1" />
     </material>
+    <xacro:wheel_link prefix="right"/>
+    <xacro:wheel_link prefix="left"/>
     <link name="base_link">
         <visual>
@@ -19,22 +32,4 @@
             <origin xyz="0 0 0.1" rpy="0 0 0" />
             <material name="blue" />
-        </visual>
-    </link>
-    <link name="right_wheel_link">
-        <visual>
-            <geometry>
-                <cylinder radius="${ wheel_radius }" length="${ wheel_length }" />
-            </geometry>
-            <origin xyz="0 0 0" rpy="${pi / 2.0} 0 0" />
-            <material name="grey" />
-        </visual>
-    </link>
-    <link name="left_wheel_link">
-        <visual>
-            <geometry>
-                <cylinder radius="${ wheel_radius }" length="${ wheel_length }" />
-            </geometry>
-            <origin xyz="0 0 0" rpy="${pi / 2.0} 0 0" />
-            <material name="grey" />
         </visual>
     </link>

Commit message: Updated wheel values

File: src/my_robot_description/urdf/my_robot.urdf.xacro (robot description, xacro)
@@ -5,5 +5,5 @@
     <xacro:property name="base_height" value="0.2" />
     <xacro:property name="wheel_radius" value="0.1" />
-    <xacro:property name="wheel_length" value="0.05" />
+    <xacro:property name="wheel_length" value="0.1" />
     <xacro:macro name="wheel_link" params="prefix">
         <link name="${prefix}_wheel_link">

Commit message: seperated xacro into multiple files

File: src/my_robot_description/urdf/my_robot.urdf.xacro (robot description, xacro)
@@ -1,70 +1,5 @@
 <?xml version="1.0"?>
 <robot name="my_robot" xmlns:xacro="http://www.ros.org/wiki/xacro">
-    <xacro:property name="base_length" value="0.6"/>
-    <xacro:property name="base_width" value="0.4" />
-    <xacro:property name="base_height" value="0.2" />
-    <xacro:property name="wheel_radius" value="0.1" />
-    <xacro:property name="wheel_length" value="0.1" />
-    <xacro:macro name="wheel_link" params="prefix">
-        <link name="${prefix}_wheel_link">
-            <visual>
-                <geometry>
-                    <cylinder radius="${wheel_radius}" length="${wheel_length}" />
-                </geometry>
-                <origin xyz="0 0 0" rpy="${pi/2.0} 0 0" />
-                <material name="grey" />
-            </visual>
-        </link>
-    </xacro:macro>
-    <material name="blue">
-        <color rgba="0 0 1 1" />
-    </material>
-    <material name="grey">
-        <color rgba="0.5 0.5 0.5 1" />
-    </material>
-    <xacro:wheel_link prefix="right"/>
-    <xacro:wheel_link prefix="left"/>
-    <link name="base_link">
-        <visual>
-            <geometry>
-                <box size="${base_length} ${base_width} ${base_height}" />
-            </geometry>
-            <origin xyz="0 0 0.1" rpy="0 0 0" />
-            <material name="blue" />
-        </visual>
-    </link>
-    <link name="caster_wheel_link">
-        <visual>
-            <geometry>
-                <sphere radius="${ wheel_radius / 2.0 }"/>
-            </geometry>
-            <origin xyz="0 0 0" rpy="0 0 0" />
-            <material name="grey" />
-        </visual>
-    </link>
-    <link name="base_footprint">
-    </link>
-    <joint name="base_base_footprint" type="fixed">
-        <parent link="base_footprint"/>
-        <child link="base_link"/>
-        <origin xyz="0 0 ${ wheel_radius }" rpy="0 0 0"/>
-    </joint>
-    <joint name="base_caster_wheel" type="continuous" >
-        <parent link="base_link" />
-        <child link="caster_wheel_link" />
-        <origin xyz="${ base_length / 4.0 } 0 ${- wheel_radius / 2.0}" rpy="0 0 0"/>
-        <axis xyz="0 1 0"/>
-    </joint>
-    <joint name="base_left_wheel" type="continuous" >
-        <parent link="base_link"/>
-        <child link="left_wheel_link"/>
-        <origin xyz="${- base_length / 4.0 } ${base_width/2.0 + wheel_length/2.0} 0" rpy="0 0 0"/>
-        <axis xyz="0 1 0" />
-    </joint>
-    <joint name="base_right_wheel" type="continuous" >
-        <parent link="base_link"/>
-        <child link="right_wheel_link"/>
-        <origin xyz="${- base_length / 4.0 } ${ -base_width / 2.0 - wheel_length/2.0} 0" rpy="0 0 0"/>
-        <axis xyz="0 1 0" />
-    </joint>
+    <xacro:include filename="common_properties.xacro" />
+    <xacro:include filename="mobile_base.xacro" />
 </robot>
